File: EAGLE/Hub Exterior/hub_exterior.brd (EAGLE design)
At the start: 49.5 x 49.5 mm, 21 parts, among them Q1 BC337, X2 LLUVIA, X4 GPS, X5 LED_ROJO, X6 BUZZER

Commit message: Update EAGLE files (hub exterior)
Connections:
- net GND: now also X1.5
Changed lines of the file:
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@@
 <wire x1="47.8125" y1="30.625" x2="47.8125" y2="12.2425" width="0.8128" layer="16"/>
 <wire x1="47.8125" y1="12.2425" x2="46.99" y2="11.42" width="0.8128" layer="16"/>
+<contactref element="X1" pad="5"/>
 <wire x1="16.6878" y1="45.085" x2="12.065" y2="32.385" width="0" layer="19" extent="1-1"/>
 </signal>
