File: KiCAD/hub_interior/hub_interior.kicad_sch (KiCad schematic)
At the start: 15 parts

Commit message: rediseño hub interior
Parts:
- C1, C2: value (none) -> 10nF; footprint (none) -> Capacitor_THT:C_Disc_D7.5mm_W2.5mm_P5.00mm
- C4: value (none) -> C-EU050-025X075; footprint (none) -> Capacitor_THT:C_Disc_D7.5mm_W2.5mm_P5.00mm
- JP1: value (none) -> PINHD-1X3; footprint (none) -> Connector_PinSocket_2.54mm:PinSocket_1x03_P2.54mm_Vertical
- LED0: value (none) -> LED_VERDE; footprint (none) -> Connector_Molex:Molex_KK-254_AE-6410-02A_1x02_P2.54mm_Vertical
- Q1: value (none) -> BC337; footprint (none) -> Package_TO_SOT_THT:TO-92
- R1: value (none) -> 10kΩ; footprint (none) -> Resistor_THT:R_Axial_DIN0207_L6.3mm_D2.5mm_P7.62mm_Horizontal
- R2: value (none) -> 1kΩ; footprint (none) -> Resistor_THT:R_Axial_DIN0207_L6.3mm_D2.5mm_P7.62mm_Horizontal
- R3, R4: value (none) -> 470Ω; footprint (none) -> Resistor_THT:R_Axial_DIN0207_L6.3mm_D2.5mm_P7.62mm_Horizontal
- RELE0, VOLTAGE0: value (none) -> 22-23-2041; footprint (none) -> Connector_Molex:Molex_KK-254_AE-6410-04A_1x04_P2.54mm_Vertical
- X1: value (none) -> F09HP; footprint (none) -> hub_interior:F09HP
- X5: value (none) -> BUZZER; footprint (none) -> Connector_Molex:Molex_KK-254_AE-6410-02A_1x02_P2.54mm_Vertical
- X6: value (none) -> LED_ROJO; footprint (none) -> Connector_Molex:Molex_KK-254_AE-6410-02A_1x02_P2.54mm_Vertical
Connections:
- net GND: no longer X1.G1, X1.G2
